File: KiCAD/MCD/MCD.kicad_pcb (KiCad board)
At the start: 2 copper layers, 3 parts, among them U1 SST39SF020A-70-4C-PHE, U2 SST39SF020A-70-4C-PHE, U3 MC68000FN

Commit message: last revision with vbcc
Parts:
- added C1: 0u1, Capacitor_SMD:C_0805_2012Metric_Pad1.18x1.45mm_HandSolder, F.Cu at (364.4, 81.2)
- added C10: 0u1, Capacitor_SMD:C_0805_2012Metric_Pad1.18x1.45mm_HandSolder, F.Cu at (358.5, 137.8)
- added C11: 0u01, Capacitor_SMD:C_0805_2012Metric_Pad1.18x1.45mm_HandSolder, F.Cu at (352.0, 153.7)
- added C12: 0u01, Capacitor_SMD:C_0805_2012Metric_Pad1.18x1.45mm_HandSolder, F.Cu at (364.5, 84.5)
- added C13: 0u01, Capacitor_SMD:C_0805_2012Metric_Pad1.18x1.45mm_HandSolder, F.Cu at (383.0, 69.7)
- added C14: 0u1, Capacitor_SMD:C_0805_2012Metric_Pad1.18x1.45mm_HandSolder, F.Cu at (361.3, 153.9)
- added C15: 0u1, Capacitor_SMD:C_0805_2012Metric_Pad1.18x1.45mm_HandSolder, F.Cu at (378.4, 66.6)
- added C16: 0u1, Capacitor_SMD:C_0805_2012Metric_Pad1.18x1.45mm_HandSolder, F.Cu at (364.4, 78.2)
- added C17: 0u1, Capacitor_SMD:C_0805_2012Metric_Pad1.18x1.45mm_HandSolder, F.Cu at (369.2, 81.4)
- added C18: 4u7, Capacitor_SMD:C_0805_2012Metric_Pad1.18x1.45mm_HandSolder, F.Cu at (320.1, 175.0)
- added C19: 4u7, Capacitor_SMD:C_0805_2012Metric_Pad1.18x1.45mm_HandSolder, F.Cu at (330.2, 171.7)
- added C2: 0u1, Capacitor_SMD:C_0805_2012Metric_Pad1.18x1.45mm_HandSolder, F.Cu at (378.1, 72.4)
- added C20: 0u1, Capacitor_SMD:C_0805_2012Metric_Pad1.18x1.45mm_HandSolder, F.Cu at (341.8, 104.9)
- added C21: 0u1, Capacitor_SMD:C_0805_2012Metric_Pad1.18x1.45mm_HandSolder, F.Cu at (342.4, 153.7)
- added C22: 0u1, Capacitor_SMD:C_0805_2012Metric_Pad1.18x1.45mm_HandSolder, F.Cu at (374.0, 78.4)
- added C23: 0u1, Capacitor_SMD:C_0805_2012Metric_Pad1.18x1.45mm_HandSolder, F.Cu at (373.3, 75.4)
- added C3: 0u01, Capacitor_SMD:C_0805_2012Metric_Pad1.18x1.45mm_HandSolder, F.Cu at (373.3, 72.4)
- added C4: 0u01, Capacitor_SMD:C_0805_2012Metric_Pad1.18x1.45mm_HandSolder, F.Cu at (378.1, 75.4)
- added C5: 0u01, Capacitor_SMD:C_0805_2012Metric_Pad1.18x1.45mm_HandSolder, F.Cu at (369.2, 78.4)
- added C6: 0u1, Capacitor_SMD:C_0805_2012Metric_Pad1.18x1.45mm_HandSolder, F.Cu at (374.0, 81.4)
- added C7: 0u01, Capacitor_SMD:C_0805_2012Metric_Pad1.18x1.45mm_HandSolder, F.Cu at (346.4, 137.8)
- added C8: 0u1, Capacitor_SMD:C_0805_2012Metric_Pad1.18x1.45mm_HandSolder, F.Cu at (350.4, 137.8)
- added C9: 0u1, Capacitor_SMD:C_0805_2012Metric_Pad1.18x1.45mm_HandSolder, F.Cu at (354.5, 137.8)
- added D1: LED, LED_SMD:LED_0805_2012Metric_Pad1.15x1.40mm_HandSolder, F.Cu at (316.8, 179.1)
- added D2: LED, LED_SMD:LED_0805_2012Metric_Pad1.15x1.40mm_HandSolder, F.Cu at (252.3, 179.9)
- added D3: LED, LED_SMD:LED_0805_2012Metric_Pad1.15x1.40mm_HandSolder, F.Cu at (256.8, 180.4)
- added D4: LED, LED_SMD:LED_0805_2012Metric_Pad1.15x1.40mm_HandSolder, F.Cu at (54.1, 213.9)
- added D5: LED, LED_SMD:LED_0805_2012Metric_Pad1.15x1.40mm_HandSolder, F.Cu at (49.0, 213.9)
- added D6: LED, LED_SMD:LED_0805_2012Metric_Pad1.15x1.40mm_HandSolder, F.Cu at (262.2, 180.6)
- added D7: LED, LED_SMD:LED_0805_2012Metric_Pad1.15x1.40mm_HandSolder, F.Cu at (267.2, 180.4)
- added D8: LED, LED_SMD:LED_0805_2012Metric_Pad1.15x1.40mm_HandSolder, F.Cu at (333.8, 175.8)
- added J1: DBUS_LOW, Imported:CON8_1X8_TU_HTS_SAI, F.Cu at (303.3, 36.8)
- added J2: DBUS_HIGH, Imported:CON8_1X8_TU_HTS_SAI, F.Cu at (329.4, 61.2)
- added J3: ABUS, Imported:CON18_2X9_TU_HTS_SAI, F.Cu at (331.0, 73.5)
- added J4: POWER, Imported:CON4_1X4_TU_HTS_SAI, F.Cu at (323.3, 49.0)
- added J5: JTAG, Imported:CON6_1X6_TU_HTS_SAI, F.Cu at (326.4, 54.6)
- added J6: Conn_01x02_Male, Imported:CON2_1X2_TU_HTS_SAI, F.Cu at (321.1, 32.3)
- added J7: DUART A, Imported:CON6_1X6_TU_HTS_SAI, F.Cu at (105.4, 108.7)
- added J8: DUART B, Imported:CON6_1X6_TU_HTS_SAI, F.Cu at (327.4, 67.3)
- added R1: 4k7, Resistor_SMD:R_0805_2012Metric_Pad1.20x1.40mm_HandSolder, F.Cu at (332.2, 120.7)
- added R10: 4k7, Resistor_SMD:R_0805_2012Metric_Pad1.20x1.40mm_HandSolder, F.Cu at (327.4, 126.5)
- added R11: 4k7, Resistor_SMD:R_0805_2012Metric_Pad1.20x1.40mm_HandSolder, F.Cu at (387.7, 68.0)
- added R12: 4k7, Resistor_SMD:R_0805_2012Metric_Pad1.20x1.40mm_HandSolder, F.Cu at (350.1, 116.9)
- added R13: 4k7, Resistor_SMD:R_0805_2012Metric_Pad1.20x1.40mm_HandSolder, F.Cu at (359.5, 110.7)
- added R14: 4k7, Resistor_SMD:R_0805_2012Metric_Pad1.20x1.40mm_HandSolder, F.Cu at (358.6, 93.2)
- added R15: 4k7, Resistor_SMD:R_0805_2012Metric_Pad1.20x1.40mm_HandSolder, F.Cu at (322.6, 132.3)
- added R16: 1k, Resistor_SMD:R_0805_2012Metric_Pad1.20x1.40mm_HandSolder, F.Cu at (316.8, 175.0)
- added R17: 1k, Resistor_SMD:R_0805_2012Metric_Pad1.20x1.40mm_HandSolder, F.Cu at (359.5, 113.7)
- added R18: 1k, Resistor_SMD:R_0805_2012Metric_Pad1.20x1.40mm_HandSolder, F.Cu at (332.2, 123.7)
- added R19: 1k, Resistor_SMD:R_0805_2012Metric_Pad1.20x1.40mm_HandSolder, F.Cu at (353.4, 99.4)
- added R2: 4k7, Resistor_SMD:R_0805_2012Metric_Pad1.20x1.40mm_HandSolder, F.Cu at (359.5, 104.8)
- added R20: 1k, Resistor_SMD:R_0805_2012Metric_Pad1.20x1.40mm_HandSolder, F.Cu at (317.8, 132.3)
- added R21: 1k, Resistor_SMD:R_0805_2012Metric_Pad1.20x1.40mm_HandSolder, F.Cu at (327.4, 129.4)
- added R22: 1k, Resistor_SMD:R_0805_2012Metric_Pad1.20x1.40mm_HandSolder, F.Cu at (353.4, 102.4)
- added R23: 1k, Resistor_SMD:R_0805_2012Metric_Pad1.20x1.40mm_HandSolder, F.Cu at (333.8, 171.7)
- added R24: 4k7, Resistor_SMD:R_0805_2012Metric_Pad1.20x1.40mm_HandSolder, F.Cu at (353.9, 93.2)
- added R3: 4k7, Resistor_SMD:R_0805_2012Metric_Pad1.20x1.40mm_HandSolder, F.Cu at (317.8, 135.2)
- added R4: 4k7, Resistor_SMD:R_0805_2012Metric_Pad1.20x1.40mm_HandSolder, F.Cu at (339.4, 114.4)
- added R5: 4k7, Resistor_SMD:R_0805_2012Metric_Pad1.20x1.40mm_HandSolder, F.Cu at (354.9, 116.6)
- added R6: 4k7, Resistor_SMD:R_0805_2012Metric_Pad1.20x1.40mm_HandSolder, F.Cu at (337.0, 117.7)
- added R7: 4k7, Resistor_SMD:R_0805_2012Metric_Pad1.20x1.40mm_HandSolder, F.Cu at (350.1, 113.9)
- added R8: 4k7, Resistor_SMD:R_0805_2012Metric_Pad1.20x1.40mm_HandSolder, F.Cu at (387.9, 65.0)
- added R9: 4k7, Resistor_SMD:R_0805_2012Metric_Pad1.20x1.40mm_HandSolder, F.Cu at (313.0, 135.2)
- added SW1: SW_Push, Button_Switch_THT:SW_PUSH_6mm, F.Cu at (328.2, 151.7)
- added U10: STM1001LWX6F, Imported:SOT-23_STM-L, F.Cu at (319.3, 99.3)
- added U4: SST39SF020A-70-4C-PHE, Imported:PDIP32_PH_SST_MCH, F.Cu at (169.1, 185.7)
- added U5: SST39SF020A-70-4C-PHE, Imported:PDIP32_PH_SST_MCH, F.Cu at (209.6, 186.4)
- added U6: XR68C681CJ-F, Imported:TO_11B1-RK-TP_3MM, F.Cu at (149.1, 123.2)
- added U7: AP2114HA-3.3TRG1, Imported:SOT-223_DIO-L, F.Cu at (325.2, 172.8)
- added U8: MAX6816EUS_T, Package_TO_SOT_SMD:SOT-143_Handsoldering, F.Cu at (310.1, 99.3)
- added U9: MC68000FN, Imported:3M_8468-11B1-RK-TP, F.Cu at (211.0, 139.8)
- added Y1: ECS-100AX-036, Imported:OSC_ECS-100AX-036, F.Cu at (126.0, 124.5)
- added Y2: ECS-100AX-080, Imported:OSC_ECS-100AX-080, F.Cu at (182.1, 136.9)
- U1: value SST39SF020A-70-4C-PHE -> XC9572XL-10VQG44C; footprint Imported:PDIP32_PH_SST_MCH -> Imported:TO_11B1-RK-TP_3MM
- U2: value SST39SF020A-70-4C-PHE -> AS6C1008-55PCN
- U3: value MC68000FN -> AS6C1008-55PCN; footprint Package_LCC:PLCC-68 -> Imported:PDIP32_PH_SST_MCH
- moved U3 72.7 mm to (115.8, 140.9)
- moved U2 69.4 mm to (139.1, 140.9)
- moved U1 59.5 mm to (181.9, 110.5)
Connections:
- U1 pad 1: unconnected-(U1-Pad1) -> CLK
- U1 pad 10: unconnected-(U1-Pad10) -> TMS
- U1 pad 11: unconnected-(U1-Pad11) -> TCK
- U1 pad 12: unconnected-(U1-Pad12) -> AS
- U1 pad 13: unconnected-(U1-Pad13) -> ROMHOE
- U1 pad 14: unconnected-(U1-Pad14) -> ROMHCE
- U1 pad 15: unconnected-(U1-Pad15) -> +3V3
- U1 pad 16: unconnected-(U1-Pad16) -> RAMLCE
- U1 pad 17: unconnected-(U1-Pad17) -> GND
- U1 pad 18: unconnected-(U1-Pad18) -> RAMLCE2
- U1 pad 19: unconnected-(U1-Pad19) -> ROMLCE
- U1 pad 2: unconnected-(U1-Pad2) -> BERR
- U1 pad 20: unconnected-(U1-Pad20) -> RAMLOE
- U1 pad 21: unconnected-(U1-Pad21) -> RAMHCE
- U1 pad 22: unconnected-(U1-Pad22) -> RAMHCE2
- U1 pad 23: unconnected-(U1-Pad23) -> ROMLOE
- U1 pad 24: unconnected-(U1-Pad24) -> TDO
- U1 pad 25: unconnected-(U1-Pad25) -> GND
- U1 pad 26: unconnected-(U1-Pad26) -> +3V3
- U1 pad 27: unconnected-(U1-Pad27) -> RAMHOE
- U1 pad 28: unconnected-(U1-Pad28) -> DUARTCS
- U1 pad 29: unconnected-(U1-Pad29) -> A20
- U1 pad 3: unconnected-(U1-Pad3) -> RESET
- U1 pad 30: unconnected-(U1-Pad30) -> A21
- U1 pad 31: unconnected-(U1-Pad31) -> A22
- U1 pad 32: unconnected-(U1-Pad32) -> A23
- U1 pad 4: unconnected-(U1-Pad4) -> GND
- U1 pad 5: unconnected-(U1-Pad5) -> HALT
- U1 pad 6: unconnected-(U1-Pad6) -> CPLD_DTACK
- U1 pad 7: unconnected-(U1-Pad7) -> UDS
- U1 pad 8: unconnected-(U1-Pad8) -> LDS
- U1 pad 9: unconnected-(U1-Pad9) -> TDI
- U2 pad 10: unconnected-(U2-Pad10) -> A3
- U2 pad 11: unconnected-(U2-Pad11) -> A2
- U2 pad 12: unconnected-(U2-Pad12) -> A1
- U2 pad 13: unconnected-(U2-Pad13) -> D0
- U2 pad 14: unconnected-(U2-Pad14) -> D1
- U2 pad 15: unconnected-(U2-Pad15) -> D2
- U2 pad 16: unconnected-(U2-Pad16) -> GND
- U2 pad 17: unconnected-(U2-Pad17) -> D3
- U2 pad 18: unconnected-(U2-Pad18) -> D4
- U2 pad 19: unconnected-(U2-Pad19) -> D5
- U2 pad 2: unconnected-(U2-Pad2) -> A17
- U2 pad 20: unconnected-(U2-Pad20) -> D6
- U2 pad 21: unconnected-(U2-Pad21) -> D7
- U2 pad 22: unconnected-(U2-Pad22) -> RAMLCE
- U2 pad 23: unconnected-(U2-Pad23) -> A11
- U2 pad 24: unconnected-(U2-Pad24) -> RAMLOE
- U2 pad 25: unconnected-(U2-Pad25) -> A12
- U2 pad 26: unconnected-(U2-Pad26) -> A10
- U2 pad 27: unconnected-(U2-Pad27) -> A9
- U2 pad 28: unconnected-(U2-Pad28) -> A14
- U2 pad 29: unconnected-(U2-Pad29) -> R/W
- U2 pad 3: unconnected-(U2-Pad3) -> A15
- U2 pad 30: unconnected-(U2-Pad30) -> RAMLCE2
- U2 pad 31: unconnected-(U2-Pad31) -> A16
- U2 pad 32: unconnected-(U2-Pad32) -> +5V
- U2 pad 4: unconnected-(U2-Pad4) -> A13
- U2 pad 5: unconnected-(U2-Pad5) -> A8
- U2 pad 6: unconnected-(U2-Pad6) -> A7
- U2 pad 7: unconnected-(U2-Pad7) -> A6
- U2 pad 8: unconnected-(U2-Pad8) -> A5
- U2 pad 9: unconnected-(U2-Pad9) -> A4
- U3 pad 10: unconnected-(U3-Pad10) -> A3
- U3 pad 11: unconnected-(U3-Pad11) -> A2
- U3 pad 12: unconnected-(U3-Pad12) -> A1
- U3 pad 13: unconnected-(U3-Pad13) -> D8
- U3 pad 14: unconnected-(U3-Pad14) -> D9
- U3 pad 15: unconnected-(U3-Pad15) -> D10
- U3 pad 16: unconnected-(U3-Pad16) -> GND
- U3 pad 17: unconnected-(U3-Pad17) -> D11
- U3 pad 18: unconnected-(U3-Pad18) -> D12
- U3 pad 19: unconnected-(U3-Pad19) -> D13
- U3 pad 2: unconnected-(U3-Pad2) -> A17
- U3 pad 20: unconnected-(U3-Pad20) -> D14
- U3 pad 21: unconnected-(U3-Pad21) -> D15
- U3 pad 22: unconnected-(U3-Pad22) -> RAMHCE
- U3 pad 23: unconnected-(U3-Pad23) -> A11
- U3 pad 24: unconnected-(U3-Pad24) -> RAMHOE
- U3 pad 25: unconnected-(U3-Pad25) -> A12
- U3 pad 26: unconnected-(U3-Pad26) -> A10
- U3 pad 27: unconnected-(U3-Pad27) -> A9
- U3 pad 28: unconnected-(U3-Pad28) -> A14
- U3 pad 29: unconnected-(U3-Pad29) -> R/W
- U3 pad 3: unconnected-(U3-Pad3) -> A15
- U3 pad 30: unconnected-(U3-Pad30) -> RAMHCE2
- U3 pad 31: unconnected-(U3-Pad31) -> A16
- U3 pad 32: unconnected-(U3-Pad32) -> +5V
- U3 pad 4: unconnected-(U3-Pad4) -> A13
- U3 pad 5: unconnected-(U3-Pad5) -> A8
- U3 pad 6: unconnected-(U3-Pad6) -> A7
- U3 pad 7: unconnected-(U3-Pad7) -> A6
- U3 pad 8: unconnected-(U3-Pad8) -> A5
- U3 pad 9: unconnected-(U3-Pad9) -> A4
Routing:
- net A18: track 0.00 -> 104.8 mm, vias 0 -> 1
- net A17: track 0.00 -> 90.3 mm, vias 0 -> 1
- net A19: track 0.00 -> 77.9 mm
- net A20: track 0.00 -> 74.3 mm
- net A21: track 0.00 -> 73.8 mm
- net A23: track 0.00 -> 66.8 mm
- net A22: track 0.00 -> 64.2 mm
- net A16: track 0.00 -> 60.2 mm, vias 0 -> 1
- net D15: track 0.00 -> 54.7 mm
- net D14: track 0.00 -> 53.6 mm, vias 0 -> 1
- net A15: track 0.00 -> 53.2 mm, vias 0 -> 1
- net A14: track 0.00 -> 52.0 mm, vias 0 -> 1
- net D13: track 0.00 -> 49.0 mm
- net D11: track 0.00 -> 45.8 mm
- net D12: track 0.00 -> 44.3 mm
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
Commit message: working on pcb
Parts:
- removed R24: 4k7, Resistor_SMD:R_0805_2012Metric_Pad1.20x1.40mm_HandSolder
- added G***: LOGO, LOGO, F.Cu at (261.3, 166.7)
- C12, C14, C15, C16, C17, C22, C23, C5, C6, C7, C9, R13: moved to B.Cu
- moved C6 263.2 mm to (121.3, 154.9), turned to 90 degrees
- moved J6 261.1 mm to (101.8, 174.2), turned to 90 degrees
- moved C5 257.0 mm to (123.8, 154.9), turned to 90 degrees
- moved C16 254.7 mm to (112.3, 114.7), turned to -90 degrees
- moved C15 246.0 mm to (134.3, 97.2), turned to 90 degrees
- moved J5 245.2 mm to (101.8, 153.2), turned to 90 degrees
- moved C12 240.3 mm to (130.8, 140.7), turned to 180 degrees
- moved J8 231.8 mm to (101.8, 120.7), turned to -90 degrees
- moved C14 231.0 mm to (130.8, 138.2), turned to 180 degrees
- moved R23 226.8 mm to (110.3, 133.2), turned to 0 degrees
- moved R17 226.6 mm to (140.8, 173.2), turned to -90 degrees
- moved C20 224.4 mm to (130.6, 180.9)
- moved U7 223.9 mm to (103.8, 138.7)
- moved D8 223.9 mm to (113.8, 134.2)
- moved C19 223.7 mm to (109.3, 136.7)
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Connections:
- D1 pad 2: Net-(D1-Pad2) -> /3V3_LED
- D8 pad 2: Net-(D8-Pad2) -> /3V3_LED
- R16 pad 2: Net-(D1-Pad2) -> /3V3_LED
- R23 pad 2: Net-(D8-Pad2) -> /3V3_LED
- U7 pad 4: +5V -> GND
Routing:
- net A18: track 104.8 -> 0.00 mm, vias 1 -> 0
- net +5V: track 27.8 -> 124.6 mm, vias 0 -> 6
- net A17: track 90.3 -> 0.00 mm, vias 1 -> 0
- net A19: track 77.9 -> 0.00 mm
- net A20: track 74.3 -> 0.00 mm
- net A21: track 73.8 -> 0.00 mm
- net A23: track 66.8 -> 0.00 mm
- net A22: track 64.2 -> 0.00 mm
- net A16: track 60.2 -> 0.00 mm, vias 1 -> 0
- net TMS: track 0.00 -> 60.0 mm, vias 0 -> 1
- net D15: track 54.7 -> 0.00 mm
- net D14: track 53.6 -> 0.00 mm, vias 1 -> 0
- net A15: track 53.2 -> 0.00 mm, vias 1 -> 0
- net TDI: track 0.00 -> 52.0 mm
- net A14: track 52.0 -> 0.00 mm, vias 1 -> 0
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Other:
- board outline added: 195 x 115 mm
- board text added: "3V3"
- board text added: "5V"
- board text added: "GEORGE YACOUBIAN LETU SP 2024 - ADD FEET - ADD VETRIUM MARKERS - 4 LAYER?"
- board text added: "HIGH RAM"
- board text added: "HIGH ROM"
- board text added: "LOW RAM"
- board text added: "LOW ROM"

Commit message: I NEED TO TAKE BRAKE
Parts:
- moved C2 6.58 mm to (238.8, 87.4)
- moved C4 6.58 mm to (236.2, 87.4)
- moved R11 6.58 mm to (237.2, 110.9)
- moved R12 6.58 mm to (241.8, 92.4)
- moved R14 6.58 mm to (237.2, 105.9)
- moved U3 6.58 mm to (218.1, 86.4)
- moved U5 6.58 mm to (248.1, 86.4)
- moved C11 6.58 mm to (266.2, 87.4)
- moved C8 6.58 mm to (268.8, 87.4)
- moved R5 6.58 mm to (267.2, 105.9)
- moved R6 6.58 mm to (267.2, 110.9)
- moved C22 0.14 mm to (166.3, 156.3)
Connections:
- U1 pad 16: RAMLCE -> RAMHCE
- U1 pad 18: RAMLCE2 -> ROMLCE
- U1 pad 19: ROMLCE -> RAMHCE2
- U1 pad 20: RAMLOE -> RAMLCE
- U1 pad 21: RAMHCE -> ROMLOE
- U1 pad 22: RAMHCE2 -> RAMLCE2
- U1 pad 23: ROMLOE -> RAMLOE
- U1 pad 28: DUARTCS -> A19
- U1 pad 44: A19 -> DUARTCS
Routing:
- net RAMHOE: track 0.00 -> 163.4 mm, vias 0 -> 2
- net ROMHOE: track 8.16 -> 158.7 mm
- net ROMHCE: track 11.2 -> 155.1 mm
- net RAMHCE2: track 21.7 -> 154.0 mm
- net RAMHCE: track 0.00 -> 126.4 mm
- net ROMLOE: track 23.0 -> 112.8 mm
- net ROMLCE: track 13.5 -> 101.3 mm
- net RAMLCE2: track 14.0 -> 101.5 mm
- net RAMLOE: track 17.5 -> 86.6 mm
- net RAMLCE: track 11.2 -> 75.3 mm
- net D1: track 0.00 -> 55.9 mm
- net D0: track 0.00 -> 55.4 mm
- net D2: track 0.00 -> 50.3 mm
- net D7: track 0.00 -> 44.4 mm
- net D6: track 0.00 -> 38.3 mm
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
Commit message: finished data bus
Parts:
- moved J3 33.2 mm to (226.8, 172.5)
- moved J2 19.1 mm to (281.6, 154.5), turned to -90 degrees
- moved J1 16.8 mm to (281.8, 133.0)
- moved C1 11.6 mm to (183.3, 88.5)
- moved C10 11.6 mm to (213.6, 88.7)
- moved C13 11.6 mm to (211.1, 88.7)
- moved C3 11.6 mm to (180.8, 88.5)
- moved R10 11.6 mm to (181.8, 107.0)
- moved R3 11.6 mm to (212.1, 107.2)
- moved R4 11.6 mm to (212.1, 112.2)
- moved R7 11.6 mm to (181.8, 112.0)
- moved R8 11.6 mm to (181.3, 93.5)
- moved U2 11.6 mm to (162.7, 87.5)
- moved U4 11.6 mm to (192.9, 87.7)
- moved C16 6.45 mm to (118.8, 114.0)
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Routing:
- net D7: track 44.4 -> 225.6 mm, vias 0 -> 3
- net D6: track 38.3 -> 218.0 mm, vias 0 -> 4
- net D15: track 0.00 -> 174.2 mm, vias 0 -> 2
- net D14: track 0.00 -> 168.3 mm, vias 0 -> 2
- net D5: track 38.3 -> 206.4 mm, vias 0 -> 3
- net D4: track 32.3 -> 196.8 mm, vias 0 -> 3
- net D13: track 0.00 -> 157.0 mm, vias 0 -> 2
- net D3: track 32.2 -> 185.8 mm, vias 0 -> 2
- net D9: track 0.00 -> 150.0 mm, vias 0 -> 2
- net D8: track 0.00 -> 148.2 mm, vias 0 -> 2
- net D12: track 0.00 -> 146.4 mm, vias 0 -> 2
- net ROMHOE: track 158.7 -> 14.8 mm
- net D10: track 0.00 -> 143.3 mm, vias 0 -> 2
- net D11: track 0.00 -> 140.8 mm, vias 0 -> 2
- net ROMHCE: track 155.1 -> 17.3 mm
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Other:
- board text added: "GEORGE YACOUBIAN LETU SP 2024 GeorgeOS Single Board Computer - ADD FEET - ADD VETRIUM MARKERS - 4 LAYER?"
- board text removed: "GEORGE YACOUBIAN LETU SP 2024 - ADD FEET - ADD VETRIUM MARKERS - 4 LAYER?"

Commit message: DO NOT CHANGE THIS BISCUIT PARAMETERS
Parts:
- R15: moved to B.Cu
- moved U7 132.0 mm to (114.7, 7.08), turned to 0 degrees
- moved R16 130.6 mm to (109.2, 13.6), turned to -90 degrees
- moved C18 128.1 mm to (112.7, 12.6), turned to 0 degrees
- moved D1 126.1 mm to (110.2, 17.1), turned to 180 degrees
- moved C19 124.3 mm to (116.7, 12.6), turned to 180 degrees
- moved R23 120.0 mm to (120.2, 13.6), turned to -90 degrees
- moved J8 119.6 mm to (132.7, 5.08), turned to 180 degrees
- moved D8 117.2 mm to (119.2, 17.1), turned to 0 degrees
- moved J7 106.4 mm to (157.7, 5.08), turned to 180 degrees
- moved J1 98.8 mm to (198.4, 79.9), turned to 180 degrees
- moved U2 93.0 mm to (233.8, 147.3), turned to 180 degrees
- moved J6 87.6 mm to (125.4, 89.8), turned to 180 degrees
- moved U3 84.4 mm to (282.6, 147.3), turned to 180 degrees
- moved J2 80.9 mm to (250.7, 79.8), turned to 180 degrees
- moved C8 68.1 mm to (237.2, 146.3), turned to 90 degrees
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Routing:
- net D7: track 225.6 -> 0.00 mm, vias 3 -> 0
- net D6: track 218.0 -> 0.17 mm, vias 4 -> 0
- net D5: track 206.4 -> 0.00 mm, vias 3 -> 0
- net D4: track 196.8 -> 0.00 mm, vias 3 -> 0
- net D3: track 185.8 -> 0.00 mm, vias 2 -> 0
- net D0: track 183.2 -> 0.00 mm, vias 2 -> 0
- net D2: track 182.1 -> 0.00 mm, vias 2 -> 0
- net D1: track 178.1 -> 0.00 mm, vias 2 -> 0
- net D15: track 174.2 -> 0.00 mm, vias 2 -> 0
- net D14: track 168.3 -> 0.00 mm, vias 2 -> 0
- net D13: track 157.0 -> 0.00 mm, vias 2 -> 0
- net D9: track 150.0 -> 0.00 mm, vias 2 -> 0
- net D8: track 148.2 -> 0.00 mm, vias 2 -> 0
- net D12: track 146.4 -> 0.00 mm, vias 2 -> 0
- net D10: track 143.3 -> 0.00 mm, vias 2 -> 0
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
Commit message: HALF OF ABUS
Parts:
- moved J3 10.3 mm to (158.7, 161.8), turned to -90 degrees
- moved C2 7.26 mm to (269.3, 145.8)
- moved C4 7.26 mm to (271.8, 145.8)
- moved R11 7.26 mm to (270.8, 122.2)
- moved R12 7.26 mm to (270.7, 140.7)
- moved R14 7.26 mm to (270.8, 127.2)
- moved U3 7.26 mm to (289.9, 146.8)
- moved C11 5.15 mm to (244.8, 145.8)
- moved C8 5.15 mm to (242.3, 145.8)
- moved R5 5.15 mm to (243.8, 127.3)
- moved R6 5.15 mm to (243.8, 122.3)
- moved U5 5.15 mm to (262.9, 146.8)
- moved C1 2.12 mm to (215.3, 146.2)
- moved C3 2.12 mm to (217.8, 146.2)
- moved R8 2.12 mm to (217.3, 141.2)
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Routing:
- net A1: track 0.00 -> 167.0 mm, vias 0 -> 2
- net A2: track 0.00 -> 154.0 mm, vias 0 -> 2
- net A3: track 0.00 -> 147.2 mm, vias 0 -> 2
- net A4: track 0.00 -> 132.8 mm, vias 0 -> 2
- net A5: track 0.00 -> 124.7 mm, vias 0 -> 2
- net A11: track 0.00 -> 108.3 mm, vias 0 -> 2
- net A6: track 0.00 -> 107.8 mm, vias 0 -> 2
- net A7: track 0.00 -> 102.2 mm, vias 0 -> 2
- net A18: track 0.00 -> 100.7 mm, vias 0 -> 2
- net A8: track 0.00 -> 90.7 mm, vias 0 -> 2
- net A10: track 0.00 -> 88.7 mm, vias 0 -> 2
- net A9: track 0.00 -> 88.6 mm, vias 0 -> 2
- net A12: track 0.00 -> 87.8 mm, vias 0 -> 2
- net A17: track 0.00 -> 87.6 mm, vias 0 -> 3
- net A13: track 0.00 -> 70.3 mm, vias 0 -> 2
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Other:
- board size 195 x 115 mm -> 219.5 x 115.5 mm

Commit message: abus done, working on dbus
Parts:
- moved G*** 233.0 mm to (115.5, 74.0)
- moved J3 4.55 mm to (156.0, 165.5), turned to 0 degrees
Routing:
- net A1: track 167.0 -> 373.2 mm, vias 2 -> 5
- net A2: track 154.0 -> 352.6 mm, vias 2 -> 5
- net A3: track 147.2 -> 338.9 mm, vias 2 -> 5
- net A4: track 132.8 -> 317.3 mm, vias 2 -> 5
- net A11: track 108.3 -> 286.4 mm, vias 2 -> 5
- net A5: track 124.7 -> 300.2 mm, vias 2 -> 5
- net A6: track 107.8 -> 281.7 mm, vias 2 -> 5
- net A7: track 102.2 -> 268.9 mm, vias 2 -> 5
- net A12: track 87.8 -> 252.7 mm, vias 2 -> 5
- net A10: track 88.7 -> 251.3 mm, vias 2 -> 5
- net A9: track 88.6 -> 248.2 mm, vias 2 -> 5
- net A8: track 90.7 -> 247.9 mm, vias 2 -> 5
- net A15: track 56.0 -> 204.0 mm, vias 2 -> 5
- net A14: track 67.9 -> 210.9 mm, vias 2 -> 5
- net A13: track 70.3 -> 212.5 mm, vias 2 -> 5
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Other:
- board size 219.5 x 115.5 mm -> 208.6 x 109.7 mm

Commit message: abus and dbus done
Routing:
- net D8: track 0.00 -> 163.9 mm, vias 0 -> 2
- net D9: track 0.00 -> 158.6 mm, vias 0 -> 2
- net D0: track 26.7 -> 160.5 mm, vias 1 -> 3
- net D1: track 44.0 -> 168.9 mm, vias 1 -> 3
- net D2: track 33.8 -> 149.9 mm, vias 1 -> 3
- net D6: track 51.9 -> 145.8 mm, vias 1 -> 3
- net D3: track 48.0 -> 139.6 mm, vias 1 -> 3
- net D5: track 56.9 -> 146.0 mm, vias 1 -> 3
- net D7: track 57.3 -> 145.2 mm, vias 1 -> 3
- net D4: track 48.6 -> 123.6 mm, vias 1 -> 3
- net D15: track 103.9 -> 145.3 mm, vias 1 -> 2
- net D14: track 104.1 -> 143.5 mm, vias 1 -> 2
- net D13: track 97.0 -> 134.5 mm, vias 1 -> 2
- net D10: track 110.3 -> 147.1 mm, vias 1 -> 2
- net D12: track 93.1 -> 128.6 mm, vias 1 -> 2
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