File: KiCAD/MCD/MCD.kicad_sch (KiCad schematic)
At the start: 65 parts

Commit message: updated GeorgeOS makefile
Parts:
- removed D?: LED, symbol Device:LED
- removed J?: Conn_01x03_Male, symbol Connector:Conn_01x03_Male
- removed R? (x5): 4k7, symbol Device:R
- added C15, C17: 0u1, symbol Device:C
- added D2, D3, D4, D5, D6, D7: LED, symbol Device:LED
- added J4: Conn_01x04_Male, symbol Connector:Conn_01x04_Male
- added J8: Conn_01x06_Male, symbol Connector:Conn_01x06_Male
- added R13, R17, R18, R19, R20, R21, R22, R9: 4k7, symbol Device:R
- gave numbers to parts that had none: 58
Connections:
- net +3V3: now also J4.1 (Pin_1); no longer J5.1 (Pin_1)
- net +5V: now also J5.1 (Pin_1), U4.31 (*WE), U5.31 (*WE), U9.23 (VPA), C15.1, C17.1, J4.2 (Pin_2), J8.3 (Pin_3), R13.1, R17.1, R18.1, R19.1, R20.1, R21.1, R22.1, R9.1; no longer U9.21 (VMA)
- net DTACK: no longer U6.10 (*DTAK), U9.10 (DTACK)
- net GND: now also U6.8 (IP0), C15.2, C17.2, D2.1 (K), D3.1 (K), D4.1 (K), D5.1 (K), D6.1 (K), D7.1 (K), J4.3 (Pin_3), J4.4 (Pin_4), J8.1 (Pin_1); no longer U1.33 (I/O/GSR), U1.34 (I/O/GTS2), U1.36 (I/O/GTS1), U1.37 (I/O_23), U1.38 (I/O_24), U1.39 (I/O_25), U1.40 (I/O_26), U1.41 (I/O_27), U1.42 (I/O_28)
- net RESET: now also U1.19 (I/O_12), R9.2; no longer U10.1 (*RST), U8.3 (OUT)
- net R/W: now also U2.29 (~{WE}), U3.29 (~{WE}); no longer U4.31 (*WE), U5.31 (*WE)
- net SW_IN: now reaches SW1.2, U8.2 (IN)
- net DUART_CLK: now reaches U6.36 (X1/CLK), Y1.8 (OUTPUT)
- net TXDB: now reaches U6.11 (RXDB)
- net TXDB: now also J8.4 (Pin_4)
- net RXDB: now reaches U6.13 (TXDB)
- net RXDB: now also J8.5 (Pin_5)
- net CTS#: no longer names the net of J7.2 (Pin_2)
- net CTS#: no longer U6.32 (OP0)
- net RAMHWE renamed CPLD_DTACK
- net CPLD_DTACK: now also U9.10 (DTACK), R13.2; no longer U3.29 (~{WE})
- removed net RAMLWE: U1.19 (I/O_12), U2.29 (~{WE})
- net RTS#: no longer names the net of J7.6 (Pin_6)
- net RTS#: no longer U6.8 (IP0)
- net RXD renamed RXDA
- net TXD renamed TXDA
- new net BRESET: U1.34 (I/O/GTS2), U8.3 (OUT)
- new net DUART_DTACK: U1.36 (I/O/GTS1), U6.10 (*DTAK)
- new net LED0: D2.2 (A), R17.2, U1.37 (I/O_23)
- new net LED1: D3.2 (A), R18.2, U1.38 (I/O_24)
- new net LED2: D4.2 (A), R19.2, U1.39 (I/O_25)
- new net LED3: D5.2 (A), R20.2, U1.40 (I/O_26)
- new net LED4: D6.2 (A), R21.2, U1.41 (I/O_27)
- new net LED5: D7.2 (A), R22.2, U1.42 (I/O_28)
- new net SRESET: U1.33 (I/O/GSR), U10.1 (*RST)
- no-connect marks 17 -> 20
Other:
- note added: "If debounced RESET OR supervisor RESET goes low, RESET => LOW"
- note added: "LED's"
- note removed: "IS THIS GOING TO CAUSE PROBLEMS WITH BEING CONNECTED TO GND?"
- moved on the sheet: J5, J7, SW1, Y2

Commit message: last revision with vbcc
Parts:
- removed R24: 4k7, symbol Device:R
- C1, C10, C11, C12, C13, C14, C15, C16, C17, C18, C19, C2, C20, C21, C22, C23, C3, C4, C5, C6, C7, C8, C9: footprint (none) -> Capacitor_SMD:C_0805_2012Metric_Pad1.18x1.45mm_HandSolder
- D1, D2, D3, D4, D5, D6, D7, D8: footprint (none) -> LED_SMD:LED_0805_2012Metric_Pad1.15x1.40mm_HandSolder
- J1: value Conn_01x08_Male -> DBUS_LOW; footprint (none) -> Imported:CON8_1X8_TU_HTS_SAI
- J2: value Conn_01x08_Male -> DBUS_HIGH; footprint (none) -> Imported:CON8_1X8_TU_HTS_SAI
- J3: value Conn_01x18_Male -> ABUS; footprint (none) -> Imported:CON18_2X9_TU_HTS_SAI
- J4: value Conn_01x04_Male -> POWER; footprint (none) -> Imported:CON4_1X4_TU_HTS_SAI
- J5: value Conn_01x06_Male -> JTAG; footprint (none) -> Imported:CON6_1X6_TU_HTS_SAI
- J6: footprint (none) -> Imported:CON2_1X2_TU_HTS_SAI
- J7: value Conn_01x06_Male -> DUART A; footprint (none) -> Imported:CON6_1X6_TU_HTS_SAI
- J8: value Conn_01x06_Male -> DUART B; footprint (none) -> Imported:CON6_1X6_TU_HTS_SAI
- R1, R10, R11, R12, R13, R14, R15, R2, R3, R4, R5, R6, R7, R8, R9: footprint (none) -> Resistor_SMD:R_0805_2012Metric_Pad1.20x1.40mm_HandSolder
- R16, R17, R18, R19, R20, R21, R22, R23: value 4k7 -> 1k; footprint (none) -> Resistor_SMD:R_0805_2012Metric_Pad1.20x1.40mm_HandSolder
- SW1: footprint (none) -> Button_Switch_THT:SW_PUSH_6mm
- U1: footprint (none) -> Imported:TO_11B1-RK-TP_3MM
- U10: footprint SOT-23_STM -> Imported:SOT-23_STM-L
- U2, U3: footprint AS6C1008-55PCN:DIP1524W45P254L4191H419Q32 -> Imported:PDIP32_PH_SST_MCH
- U4, U5: footprint PDIP32_PH_SST_MCH -> Imported:PDIP32_PH_SST_MCH
- U6: footprint PLCC-44 -> Imported:TO_11B1-RK-TP_3MM
- U7: footprint SOT-223_DIO -> Imported:SOT-223_DIO-L
- U8: footprint MAX6816EUS_T:SOT192P237X122-4N -> Package_TO_SOT_SMD:SOT-143_Handsoldering
- U9: footprint Package_LCC:PLCC-68 -> Imported:3M_8468-11B1-RK-TP
- Y1: footprint ECS-100AX-036:OSC_ECS-100AX-036 -> Imported:OSC_ECS-100AX-036
- Y2: footprint ECS-100AX-080:OSC_ECS-100AX-080 -> Imported:OSC_ECS-100AX-080
Connections:
- net +3V3: now also J5.1 (Pin_1)
- net +5V: no longer J5.1 (Pin_1)
- net AS: now also U1.12 (I/O_7); no longer U1.2 (I/O_1)
- net BERR: now also U1.2 (I/O_1); no longer U1.7 (I/O_5)
- net CPLD_DTACK: now also U1.6 (I/O_4); no longer U1.23 (I/O_16)
- net GND: no longer U1.43 (I/O/GCK1), U6.3 (IP3), U6.40 (IP2), U6.42 (IP5), U6.43 (IP4), U6.5 (IP1), U6.8 (IP0)
- net HALT: now also U1.5 (I/O_3); no longer U1.6 (I/O_4)
- net LDS: now also U1.8 (I/O_6); no longer U1.5 (I/O_3)
- net RESET: now also U1.3 (I/O_2); no longer U1.19 (I/O_12)
- net ROMLCE: now also U1.19 (I/O_12); no longer U1.12 (I/O_7)
- net ROMLOE: now also U1.23 (I/O_16); no longer U1.8 (I/O_6)
- net UDS: now also U1.7 (I/O_5); no longer U1.3 (I/O_2)
- no-connect marks 20 -> 27
Other:
- note added: "HIGH"
- note added: "LOW"

Commit message: working on pcb
Connections:
- net +5V: no longer U7.4 (EPAD)
- net GND: now also U7.4 (EPAD)
- net 3V3_LED: now reaches D8.2 (A), R23.2
- net 3V3_LED: now also D1.2 (A), R16.2
Changed lines of the file:
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@@
   (junction (at 124.46 206.375) (diameter 0) (color 0 0 0 0)
   )
+  (junction (at 260.985 45.085) (diameter 0) (color 0 0 0 0)
+  )
   (junction (at 107.95 238.125) (diameter 0) (color 0 0 0 0)
   )
@@
   (junction (at 244.475 40.005) (diameter 0) (color 0 0 0 0)
   )
-  (junction (at 257.81 40.005) (diameter 0) (color 0 0 0 0)
-  )
   (junction (at 287.02 192.405) (diameter 0) (color 0 0 0 0)
   )
@@
     (stroke (width 0) (type default) (color 0 0 0 0))
   )
-  (wire (pts (xy 257.81 42.545) (xy 257.81 40.005))
-    (stroke (width 0) (type default) (color 0 0 0 0))
-  )
   (wire (pts (xy 389.89 118.11) (xy 395.605 118.11))
     (stroke (width 0) (type default) (color 0 0 0 0))
@@
     (stroke (width 0) (type default) (color 0 0 0 0))
   )
-  (wire (pts (xy 252.73 40.005) (xy 257.81 40.005))
+  (wire (pts (xy 252.73 40.005) (xy 260.985 40.005))
     (stroke (width 0) (type default) (color 0 0 0 0))
   )
@@
     (stroke (width 0) (type default) (color 0 0 0 0))
   )
-  (wire (pts (xy 260.985 42.545) (xy 257.81 42.545))
-    (stroke (width 0) (type default) (color 0 0 0 0))
-  )
   (wire (pts (xy 98.425 36.83) (xy 103.505 36.83))
     (stroke (width 0) (type default) (color 0 0 0 0))
@@
     (stroke (width 0) (type default) (color 0 0 0 0))
   )
-  (wire (pts (xy 257.81 40.005) (xy 260.985 40.005))
-    (stroke (width 0) (type default) (color 0 0 0 0))
-  )
   (bus (pts (xy 202.565 180.34) (xy 202.565 182.88))
     (stroke (width 0) (type default) (color 0 0 0 0))
@@
     (stroke (width 0) (type default) (color 0 0 0 0))
   )
+  (wire (pts (xy 260.985 42.545) (xy 260.985 45.085))
+    (stroke (width 0) (type default) (color 0 0 0 0))
+  )
   (wire (pts (xy 143.51 37.465) (xy 157.48 37.465))
     (stroke (width 0) (type default) (color 0 0 0 0))
@@
     (effects (font (size 1.27 1.27)) (justify left bottom))
   )
+  (label "3V3_LED" (at 311.15 50.165 0)
+    (effects (font (size 1.27 1.27)) (justify left bottom))
+  )
+  (label "3V3_LED" (at 252.73 50.165 180)
+    (effects (font (size 1.27 1.27)) (justify right bottom))
+  )
   (label "D12" (at 391.795 194.31 0)

Commit message: I NEED TO TAKE BRAKE
Connections:
- net A19: now also U1.28 (I/O_18); no longer U1.44 (I/O/GCK2)
- net DUARTCS: now also U1.44 (I/O/GCK2); no longer U1.28 (I/O_18)
- net RAMHCE: now also U1.16 (I/O_10); no longer U1.21 (I/O_14)
- net RAMHCE2: now also U1.19 (I/O_12); no longer U1.22 (I/O_15)
- net RAMLCE: now also U1.20 (I/O_13); no longer U1.16 (I/O_10)
- net RAMLCE2: now also U1.22 (I/O_15); no longer U1.18 (I/O_11)
- net RAMLOE: now also U1.23 (I/O_16); no longer U1.20 (I/O_13)
- net ROMLCE: now also U1.18 (I/O_11); no longer U1.19 (I/O_12)
- net ROMLOE: now also U1.21 (I/O_14); no longer U1.23 (I/O_16)

Commit message: KICAD WAS GOOFY! anyuways decode bus is done, routing control bus
Connections:
- net A19: now also U1.36 (I/O/GTS1); no longer U1.28 (I/O_18)
- net A20: now also U1.34 (I/O/GTS2); no longer U1.29 (I/O_19)
- net A21: now also U1.31 (I/O_21); no longer U1.30 (I/O_20)
- net A22: now also U1.29 (I/O_19); no longer U1.31 (I/O_21)
- net AS: now also U1.42 (I/O_28); no longer U1.12 (I/O_7)
- net BERR: now also U1.33 (I/O/GSR); no longer U1.2 (I/O_1)
- net BRESET: now also U1.18 (I/O_11); no longer U1.34 (I/O/GTS2)
- net CLK: now also U1.44 (I/O/GCK2); no longer U1.1 (I/O/GCK3)
- net CPLD_DTACK: now also U1.38 (I/O_24); no longer U1.6 (I/O_4)
- net DUARTCS: now also U1.1 (I/O/GCK3); no longer U1.44 (I/O/GCK2)
- net DUART_DTACK: now also U1.2 (I/O_1); no longer U1.36 (I/O/GTS1)
- net HALT: now also U1.39 (I/O_25); no longer U1.5 (I/O_3)
- net LDS: now also U1.41 (I/O_27); no longer U1.8 (I/O_6)
- net LED0: now also U1.20 (I/O_13); no longer U1.37 (I/O_23)
- net LED1: now also U1.22 (I/O_15); no longer U1.38 (I/O_24)
- net LED2: now also U1.23 (I/O_16); no longer U1.39 (I/O_25)
- net LED3: now also U1.27 (I/O_17); no longer U1.40 (I/O_26)
- net LED4: now also U1.28 (I/O_18); no longer U1.41 (I/O_27)
- net LED5: now also U1.30 (I/O_20); no longer U1.42 (I/O_28)
- net RAMHOE: now also U1.12 (I/O_7); no longer U1.27 (I/O_17)
- net RAMLCE: now also U1.5 (I/O_3); no longer U1.20 (I/O_13)
- net RAMLCE2: now also U1.7 (I/O_5); no longer U1.22 (I/O_15)
- net RAMLOE: now also U1.8 (I/O_6); no longer U1.23 (I/O_16)
- net RESET: now also U1.37 (I/O_23); no longer U1.3 (I/O_2)
- net ROMLCE: now also U1.3 (I/O_2); no longer U1.18 (I/O_11)
- net ROMLOE: now also U1.6 (I/O_4); no longer U1.21 (I/O_14)
- net SRESET: now also U1.21 (I/O_14); no longer U1.33 (I/O/GSR)
- net UDS: now also U1.40 (I/O_26); no longer U1.7 (I/O_5)

Commit message: everything but power connected
Connections:
- net DTACK is gone; now on net CPLD_DTACK: J6.2 (Pin_2)
- net LED0: now also U1.3 (I/O_2); no longer U1.20 (I/O_13)
- net LED1: now also U1.5 (I/O_3); no longer U1.22 (I/O_15)
- net LED2: now also U1.6 (I/O_4); no longer U1.23 (I/O_16)
- net LED3: now also U1.8 (I/O_6); no longer U1.27 (I/O_17)
- net LED4: now also U1.7 (I/O_5); no longer U1.28 (I/O_18)
- net LED5: now also U1.12 (I/O_7); no longer U1.30 (I/O_20)
- net RAMHCE2: now also U1.14 (I/O_9); no longer U1.19 (I/O_12)
- net RAMHOE: now also U1.13 (I/O_8); no longer U1.12 (I/O_7)
- net RAMLCE: now also U1.27 (I/O_17); no longer U1.5 (I/O_3)
- net RAMLCE2: now also U1.22 (I/O_15); no longer U1.7 (I/O_5)
- net RAMLOE: now also U1.23 (I/O_16); no longer U1.8 (I/O_6)
- net ROMHCE: now also U1.20 (I/O_13); no longer U1.14 (I/O_9)
- net ROMHOE: now also U1.19 (I/O_12); no longer U1.13 (I/O_8)
- net ROMLCE: now also U1.30 (I/O_20); no longer U1.3 (I/O_2)
- net ROMLOE: now also U1.28 (I/O_18); no longer U1.6 (I/O_4)
Changed lines of the file:
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@@
     )
   )
-  (global_label "DTACK" (shape input) (at 286.385 257.81 0) (fields_autoplaced)
+  (global_label "CPLD_DTACK" (shape input) (at 286.385 257.81 0) (fields_autoplaced)
     (effects (font (size 1.27 1.27)) (justify left))
-    (property "Intersheet References" "${INTERSHEET_REFS}" (id 0) (at 294.6643 257.7306 0)
+    (property "Intersheet References" "${INTERSHEET_REFS}" (id 0) (at 300.47 257.7306 0)
       (effects (font (size 1.27 1.27)) (justify left) hide)
     )

Commit message: FINISHED!!! (I THINK)
Parts:
- added FID1, FID2, FID3, FID4, FID5, FID6: Fiducial, Fiducial:Fiducial_1.5mm_Mask3mm, symbol Mechanical:Fiducial
Connections:
- net 3V3_LED: no longer D1.2 (A), R16.2
- new net 5V_LED: D1.2 (A), R16.2
Other:
- note added: "Fiducial Markers"
Changed lines of the file:
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@@
     (stroke (width 0) (type default) (color 0 0 0 0))
   )
+  (polyline (pts (xy 160.655 246.38) (xy 90.17 246.38))
+    (stroke (width 0) (type default) (color 0 0 0 0))
+  )
   (bus (pts (xy 220.98 70.485) (xy 220.98 73.025))
     (stroke (width 0) (type default) (color 0 0 0 0))
@@
     (stroke (width 0) (type default) (color 0 0 0 0))
   )
+  (polyline (pts (xy 90.17 246.38) (xy 90.17 267.335))
+    (stroke (width 0) (type default) (color 0 0 0 0))
+  )
   (bus (pts (xy 243.205 246.38) (xy 245.745 246.38))
     (stroke (width 0) (type default) (color 0 0 0 0))
@@
     (effects (font (size 1.27 1.27)) (justify left bottom))
   )
+  (text "Fiducial Markers" (at 118.745 254.635 0)
+    (effects (font (size 3 3) (thickness 0.6) bold) (justify left bottom))
+  )
   (text "FROM DUART TXD -->" (at 273.05 106.68 0)
     (effects (font (size 1.27 1.27)) (justify left bottom))
@@
     (effects (font (size 1.27 1.27)) (justify left bottom))
   )
-  (label "3V3_LED" (at 252.73 50.165 180)
+  (label "5V_LED" (at 252.73 50.165 180)
     (effects (font (size 1.27 1.27)) (justify right bottom))
   )
@@
     (pin "9")
   )
+  (symbol (lib_id "Mechanical:Fiducial") (at 92.71 252.095 0) (unit 1)
+    (in_bom yes) (on_board yes) (fields_autoplaced)
+    (property "Reference" "FID4" (id 0) (at 95.885 250.8249 0)
+      (effects (font (size 1.27 1.27)) (justify left))
+    )
+    (property "Value" "Fiducial" (id 1) (at 95.885 253.3649 0)
+      (effects (font (size 1.27 1.27)) (justify left))
+    )
+    (property "Footprint" "Fiducial:Fiducial_1.5mm_Mask3mm" (id 2) (at 92.71 252.095 0)
+      (effects (font (size 1.27 1.27)) hide)
+    )
+    (property "Datasheet" "~" (id 3) (at 92.71 252.095 0)
+      (effects (font (size 1.27 1.27)) hide)
+    )
+  )
   (symbol (lib_name "SST39SF020A-70-4C-PHE_1") (lib_id "Imported:SST39SF020A-70-4C-PHE") (at 173.355 90.17 0) (unit 1)
     (in_bom yes) (on_board yes) (fields_autoplaced)
@@
     (pin "2")
   )
+  (symbol (lib_id "Mechanical:Fiducial") (at 92.71 263.525 0) (unit 1)
+    (in_bom yes) (on_board yes) (fields_autoplaced)
+    (property "Reference" "FID6" (id 0) (at 95.885 262.2549 0)
+      (effects (font (size 1.27 1.27)) (justify left))
+    )
+    (property "Value" "Fiducial" (id 1) (at 95.885 264.7949 0)
+      (effects (font (size 1.27 1.27)) (justify left))
+    )
+    (property "Footprint" "Fiducial:Fiducial_1.5mm_Mask3mm" (id 2) (at 92.71 263.525 0)
+      (effects (font (size 1.27 1.27)) hide)
+    )
+    (property "Datasheet" "~" (id 3) (at 92.71 263.525 0)
+      (effects (font (size 1.27 1.27)) hide)
+    )
+  )
   (symbol (lib_id "power:GND") (at 83.185 245.745 0) (mirror y) (unit 1)
     (in_bom yes) (on_board yes)
@@
     (pin "6")
   )
+  (symbol (lib_id "Mechanical:Fiducial") (at 92.71 257.81 0) (unit 1)
+    (in_bom yes) (on_board yes) (fields_autoplaced)
+    (property "Reference" "FID5" (id 0) (at 95.25 256.5399 0)
+      (effects (font (size 1.27 1.27)) (justify left))
+    )
+    (property "Value" "Fiducial" (id 1) (at 95.25 259.0799 0)
+      (effects (font (size 1.27 1.27)) (justify left))
+    )
+    (property "Footprint" "Fiducial:Fiducial_1.5mm_Mask3mm" (id 2) (at 92.71 257.81 0)
+      (effects (font (size 1.27 1.27)) hide)
+    )
+    (property "Datasheet" "~" (id 3) (at 92.71 257.81 0)
+      (effects (font (size 1.27 1.27)) hide)
+    )
+  )
+  (symbol (lib_id "Mechanical:Fiducial") (at 107.315 252.095 0) (unit 1)
+    (in_bom yes) (on_board yes) (fields_autoplaced)
+    (property "Reference" "FID1" (id 0) (at 110.49 250.8249 0)
+      (effects (font (size 1.27 1.27)) (justify left))
+    )
+    (property "Value" "Fiducial" (id 1) (at 110.49 253.3649 0)
+      (effects (font (size 1.27 1.27)) (justify left))
+    )
+    (property "Footprint" "Fiducial:Fiducial_1.5mm_Mask3mm" (id 2) (at 107.315 252.095 0)
+      (effects (font (size 1.27 1.27)) hide)
+    )
+    (property "Datasheet" "~" (id 3) (at 107.315 252.095 0)
+      (effects (font (size 1.27 1.27)) hide)
+    )
+  )
   (symbol (lib_id "Connector:Conn_01x02_Male") (at 281.305 255.27 0) (unit 1)
     (in_bom yes) (on_board yes)
@@
     (pin "1")
   )
+  (symbol (lib_id "Mechanical:Fiducial") (at 107.315 263.525 0) (unit 1)
+    (in_bom yes) (on_board yes) (fields_autoplaced)
+    (property "Reference" "FID3" (id 0) (at 110.49 262.2549 0)
+      (effects (font (size 1.27 1.27)) (justify left))
+    )
+    (property "Value" "Fiducial" (id 1) (at 110.49 264.7949 0)
+      (effects (font (size 1.27 1.27)) (justify left))
+    )
+    (property "Footprint" "Fiducial:Fiducial_1.5mm_Mask3mm" (id 2) (at 107.315 263.525 0)
+      (effects (font (size 1.27 1.27)) hide)
+    )
+    (property "Datasheet" "~" (id 3) (at 107.315 263.525 0)
+      (effects (font (size 1.27 1.27)) hide)
+    )
+  )
+  (symbol (lib_id "Mechanical:Fiducial") (at 107.315 257.81 0) (unit 1)
+    (in_bom yes) (on_board yes) (fields_autoplaced)
+    (property "Reference" "FID2" (id 0) (at 109.855 256.5399 0)
+      (effects (font (size 1.27 1.27)) (justify left))
+    )
+    (property "Value" "Fiducial" (id 1) (at 109.855 259.0799 0)
+      (effects (font (size 1.27 1.27)) (justify left))
+    )
+    (property "Footprint" "Fiducial:Fiducial_1.5mm_Mask3mm" (id 2) (at 107.315 257.81 0)
+      (effects (font (size 1.27 1.27)) hide)
+    )
+    (property "Datasheet" "~" (id 3) (at 107.315 257.81 0)
+      (effects (font (size 1.27 1.27)) hide)
+    )
+  )
   (symbol (lib_id "Connector:Conn_01x08_Male") (at 163.195 251.46 0) (unit 1)
     (in_bom yes) (on_board yes)
@@
       (reference "D8") (unit 1) (value "LED") (footprint "LED_SMD:LED_0805_2012Metric_Pad1.15x1.40mm_HandSolder")
     )
+    (path "/94870077-11f0-46cd-9b00-3610a9c78eac"
+      (reference "FID1") (unit 1) (value "Fiducial") (footprint "Fiducial:Fiducial_1.5mm_Mask3mm")
+    )
+    (path "/fa1909f9-387a-4e1c-ab95-ac26baf5316d"
+      (reference "FID2") (unit 1) (value "Fiducial") (footprint "Fiducial:Fiducial_1.5mm_Mask3mm")
+    )
+    (path "/f54f50d2-50f0-4b25-8c59-fefc8fcf5c3b"
+      (reference "FID3") (unit 1) (value "Fiducial") (footprint "Fiducial:Fiducial_1.5mm_Mask3mm")
+    )
+    (path "/0cbe6fd8-5824-41c5-aa8b-5843bd7d8e06"
+      (reference "FID4") (unit 1) (value "Fiducial") (footprint "Fiducial:Fiducial_1.5mm_Mask3mm")
+    )
+    (path "/90b02067-bbc0-4431-93bf-492d98dd19c2"
+      (reference "FID5") (unit 1) (value "Fiducial") (footprint "Fiducial:Fiducial_1.5mm_Mask3mm")
+    )
+    (path "/871b13b5-562b-42ad-bc82-6ce0488ff442"
+      (reference "FID6") (unit 1) (value "Fiducial") (footprint "Fiducial:Fiducial_1.5mm_Mask3mm")
+    )
     (path "/fcb57dc0-a59b-4030-afe4-35c0fb529eb9"
