File: KiCAD/MCD/MCD.kicad_sch (KiCad schematic)
At the start: 81 parts, among them J1 DBUS_LOW, J2 DBUS_HIGH, J3 ABUS, J4 POWER, J5 JTAG, J6 Conn_01x02_Male, J7 DUART A, J8 DUART B, SW1 SW_Push, U1 XC9572XL-10VQG44C, U10 STM1001LWX6F, U2 AS6C1008-55PCN, U3 AS6C1008-55PCN, U4 SST39SF020A-70-4C-PHE, U5 SST39SF020A-70-4C-PHE, U6 XR68C681CJ-F, U7 AP2114HA-3.3TRG1, U8 MAX6816EUS_T, U9 MC68000FN, Y1 ECS-100AX-036, Y2 ECS-100AX-080

Commit message: board and parts ordered
Parts:
- removed FID1, FID2, FID3, FID4, FID5, FID6: Fiducial, Fiducial:Fiducial_1.5mm_Mask3mm, symbol Mechanical:Fiducial
Other:
- note removed: "Fiducial Markers"
Changed lines of the file:
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@@
     (stroke (width 0) (type default) (color 0 0 0 0))
   )
-  (polyline (pts (xy 160.655 246.38) (xy 90.17 246.38))
-    (stroke (width 0) (type default) (color 0 0 0 0))
-  )
   (bus (pts (xy 220.98 70.485) (xy 220.98 73.025))
     (stroke (width 0) (type default) (color 0 0 0 0))
@@
     (stroke (width 0) (type default) (color 0 0 0 0))
   )
-  (polyline (pts (xy 90.17 246.38) (xy 90.17 267.335))
-    (stroke (width 0) (type default) (color 0 0 0 0))
-  )
   (bus (pts (xy 243.205 246.38) (xy 245.745 246.38))
     (stroke (width 0) (type default) (color 0 0 0 0))
@@
     (effects (font (size 1.27 1.27)) (justify left bottom))
   )
-  (text "Fiducial Markers" (at 118.745 254.635 0)
-    (effects (font (size 3 3) (thickness 0.6) bold) (justify left bottom))
-  )
   (text "FROM DUART TXD -->" (at 273.05 106.68 0)
     (effects (font (size 1.27 1.27)) (justify left bottom))
@@
     (pin "9")
   )
-  (symbol (lib_id "Mechanical:Fiducial") (at 92.71 252.095 0) (unit 1)
-    (in_bom yes) (on_board yes) (fields_autoplaced)
-    (property "Reference" "FID4" (id 0) (at 95.885 250.8249 0)
-      (effects (font (size 1.27 1.27)) (justify left))
-    )
-    (property "Value" "Fiducial" (id 1) (at 95.885 253.3649 0)
-      (effects (font (size 1.27 1.27)) (justify left))
-    )
-    (property "Footprint" "Fiducial:Fiducial_1.5mm_Mask3mm" (id 2) (at 92.71 252.095 0)
-      (effects (font (size 1.27 1.27)) hide)
-    )
-    (property "Datasheet" "~" (id 3) (at 92.71 252.095 0)
-      (effects (font (size 1.27 1.27)) hide)
-    )
-  )
   (symbol (lib_name "SST39SF020A-70-4C-PHE_1") (lib_id "Imported:SST39SF020A-70-4C-PHE") (at 173.355 90.17 0) (unit 1)
     (in_bom yes) (on_board yes) (fields_autoplaced)
@@
     (pin "2")
   )
-  (symbol (lib_id "Mechanical:Fiducial") (at 92.71 263.525 0) (unit 1)
-    (in_bom yes) (on_board yes) (fields_autoplaced)
-    (property "Reference" "FID6" (id 0) (at 95.885 262.2549 0)
-      (effects (font (size 1.27 1.27)) (justify left))
-    )
-    (property "Value" "Fiducial" (id 1) (at 95.885 264.7949 0)
-      (effects (font (size 1.27 1.27)) (justify left))
-    )
-    (property "Footprint" "Fiducial:Fiducial_1.5mm_Mask3mm" (id 2) (at 92.71 263.525 0)
-      (effects (font (size 1.27 1.27)) hide)
-    )
-    (property "Datasheet" "~" (id 3) (at 92.71 263.525 0)
-      (effects (font (size 1.27 1.27)) hide)
-    )
-  )
   (symbol (lib_id "power:GND") (at 83.185 245.745 0) (mirror y) (unit 1)
     (in_bom yes) (on_board yes)
@@
     (pin "6")
   )
-  (symbol (lib_id "Mechanical:Fiducial") (at 92.71 257.81 0) (unit 1)
-    (in_bom yes) (on_board yes) (fields_autoplaced)
-    (property "Reference" "FID5" (id 0) (at 95.25 256.5399 0)
-      (effects (font (size 1.27 1.27)) (justify left))
-    )
-    (property "Value" "Fiducial" (id 1) (at 95.25 259.0799 0)
-      (effects (font (size 1.27 1.27)) (justify left))
-    )
-    (property "Footprint" "Fiducial:Fiducial_1.5mm_Mask3mm" (id 2) (at 92.71 257.81 0)
-      (effects (font (size 1.27 1.27)) hide)
-    )
-    (property "Datasheet" "~" (id 3) (at 92.71 257.81 0)
-      (effects (font (size 1.27 1.27)) hide)
-    )
-  )
-  (symbol (lib_id "Mechanical:Fiducial") (at 107.315 252.095 0) (unit 1)
-    (in_bom yes) (on_board yes) (fields_autoplaced)
-    (property "Reference" "FID1" (id 0) (at 110.49 250.8249 0)
-      (effects (font (size 1.27 1.27)) (justify left))
-    )
-    (property "Value" "Fiducial" (id 1) (at 110.49 253.3649 0)
-      (effects (font (size 1.27 1.27)) (justify left))
-    )
-    (property "Footprint" "Fiducial:Fiducial_1.5mm_Mask3mm" (id 2) (at 107.315 252.095 0)
-      (effects (font (size 1.27 1.27)) hide)
-    )
-    (property "Datasheet" "~" (id 3) (at 107.315 252.095 0)
-      (effects (font (size 1.27 1.27)) hide)
-    )
-  )
   (symbol (lib_id "Connector:Conn_01x02_Male") (at 281.305 255.27 0) (unit 1)
     (in_bom yes) (on_board yes)
@@
     (pin "1")
   )
-  (symbol (lib_id "Mechanical:Fiducial") (at 107.315 263.525 0) (unit 1)
-    (in_bom yes) (on_board yes) (fields_autoplaced)
-    (property "Reference" "FID3" (id 0) (at 110.49 262.2549 0)
-      (effects (font (size 1.27 1.27)) (justify left))
-    )
-    (property "Value" "Fiducial" (id 1) (at 110.49 264.7949 0)
-      (effects (font (size 1.27 1.27)) (justify left))
-    )
-    (property "Footprint" "Fiducial:Fiducial_1.5mm_Mask3mm" (id 2) (at 107.315 263.525 0)
-      (effects (font (size 1.27 1.27)) hide)
-    )
-    (property "Datasheet" "~" (id 3) (at 107.315 263.525 0)
-      (effects (font (size 1.27 1.27)) hide)
-    )
-  )
-  (symbol (lib_id "Mechanical:Fiducial") (at 107.315 257.81 0) (unit 1)
-    (in_bom yes) (on_board yes) (fields_autoplaced)
-    (property "Reference" "FID2" (id 0) (at 109.855 256.5399 0)
-      (effects (font (size 1.27 1.27)) (justify left))
-    )
-    (property "Value" "Fiducial" (id 1) (at 109.855 259.0799 0)
-      (effects (font (size 1.27 1.27)) (justify left))
-    )
-    (property "Footprint" "Fiducial:Fiducial_1.5mm_Mask3mm" (id 2) (at 107.315 257.81 0)
-      (effects (font (size 1.27 1.27)) hide)
-    )
-    (property "Datasheet" "~" (id 3) (at 107.315 257.81 0)
-      (effects (font (size 1.27 1.27)) hide)
-    )
-  )
   (symbol (lib_id "Connector:Conn_01x08_Male") (at 163.195 251.46 0) (unit 1)
     (in_bom yes) (on_board yes)
@@
       (reference "D8") (unit 1) (value "LED") (footprint "LED_SMD:LED_0805_2012Metric_Pad1.15x1.40mm_HandSolder")
     )
-    (path "/94870077-11f0-46cd-9b00-3610a9c78eac"
-      (reference "FID1") (unit 1) (value "Fiducial") (footprint "Fiducial:Fiducial_1.5mm_Mask3mm")
-    )
-    (path "/fa1909f9-387a-4e1c-ab95-ac26baf5316d"
-      (reference "FID2") (unit 1) (value "Fiducial") (footprint "Fiducial:Fiducial_1.5mm_Mask3mm")
-    )
-    (path "/f54f50d2-50f0-4b25-8c59-fefc8fcf5c3b"
-      (reference "FID3") (unit 1) (value "Fiducial") (footprint "Fiducial:Fiducial_1.5mm_Mask3mm")
-    )
-    (path "/0cbe6fd8-5824-41c5-aa8b-5843bd7d8e06"
-      (reference "FID4") (unit 1) (value "Fiducial") (footprint "Fiducial:Fiducial_1.5mm_Mask3mm")
-    )
-    (path "/90b02067-bbc0-4431-93bf-492d98dd19c2"
-      (reference "FID5") (unit 1) (value "Fiducial") (footprint "Fiducial:Fiducial_1.5mm_Mask3mm")
-    )
-    (path "/871b13b5-562b-42ad-bc82-6ce0488ff442"
-      (reference "FID6") (unit 1) (value "Fiducial") (footprint "Fiducial:Fiducial_1.5mm_Mask3mm")
-    )
     (path "/fcb57dc0-a59b-4030-afe4-35c0fb529eb9"
