File: KiCAD/MCD/MCD.kicad_sch (KiCad schematic)
At the start: 75 parts, among them J1 DBUS_LOW, J2 DBUS_HIGH, J3 ABUS, J4 POWER, J5 JTAG, J6 Conn_01x02_Male, J7 DUART A, J8 DUART B, SW1 SW_Push, U1 XC9572XL-10VQG44C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

Commit message: changed xc9572xl schematic symbol from vq44 to pc44
Parts:
- removed U1: XC9572XL-10VQG44C, Imported:TO_11B1-RK-TP_3MM, symbol Imported:XC9572XL-10VQG44C
- added U?: XC9572XL-PC44, symbol Imported:XC9572XL-PC44
- U8: footprint Package_TO_SOT_SMD:SOT-143_Handsoldering -> Package_TO_SOT_SMD:SOT-143R_Reverse_Handsoldering
Connections:
- net +3V3: now also U?.21 (VCCINT_3.3V_1), U?.32 (VCCIO_2.5V/3.3V), U?.41 (VCCINT_3.3V_2)
- net A19: now also U?.13 (I/O_9)
- net A20: now also U?.14 (I/O_10)
- net A21: now also U?.18 (I/O_11)
- net A22: now also U?.19 (I/O_12)
- net A23: now also U?.20 (I/O_13)
- net AS: now also U?.22 (I/O_14)
- net BERR: now also U?.27 (I/O_18)
- net BRESET: now also U?.2 (I/O_2)
- net CLK: now also U?.7 (I/O/GCK3)
- net CPLD_DTACK: now also U?.39 (I/O/GSR)
- net DUARTCS: now also U?.42 (I/O/GTS1)
- net DUART_DTACK: now also U?.3 (I/O_3)
- net GND: now also U?.10 (GND_1), U?.23 (GND_2), U?.31 (GND_3)
- net HALT: now also U?.26 (I/O_17)
- net LDS: now also U?.25 (I/O_16)
- net LED0: now also U?.4 (I/O_4)
- net LED1: now also U?.5 (I/O/GCK1)
- net LED2: now also U?.6 (I/O/GCK2)
- net LED3: now also U?.8 (I/O_5)
- net LED4: now also U?.9 (I/O_6)
- net LED5: now also U?.11 (I/O_7)
- net RAMHCE: now also U?.43 (I/O_27)
- net RAMHCE2: now also U?.44 (I/O_28)
- net RAMHOE: now also U?.40 (I/O/GTS2)
- net RAMLCE: now also U?.35 (I/O_23)
- net RAMLCE2: now also U?.36 (I/O_24)
- net RAMLOE: now also U?.38 (I/O_26)
- net RESET: now also U?.37 (I/O_25)
- net ROMHCE: now also U?.34 (I/O_22)
- net ROMHOE: now also U?.33 (I/O_21)
- net ROMLCE: now also U?.29 (I/O_20)
- net ROMLOE: now also U?.28 (I/O_19)
- net SRESET: now also U?.1 (I/O_1)
- net TCK: now also U?.17 (TCK)
- net TDI: now also U?.15 (TDI)
- net TDO: now also U?.30 (TDO)
- net TMS: now also U?.16 (TMS)
- net UDS: now also U?.24 (I/O_15)
Other:
- note added: "PULL UP DUART DTACK?"
Changed lines of the file:
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@@
     (effects (font (size 1.27 1.27) (thickness 0.4) bold) (justify left bottom))
   )
+  (text "PULL UP DUART DTACK?" (at 176.53 189.865 0)
+    (effects (font (size 1.27 1.27)) (justify left bottom))
+  )
   (text "FROM DUART TXD -->" (at 273.05 132.08 0)
     (effects (font (size 1.27 1.27)) (justify left bottom))
@@
     (pin "1")
   )
-  (symbol (lib_id "Imported:XC9572XL-10VQG44C") (at 27.94 189.865 0) (unit 1)
-    (in_bom yes) (on_board yes) (fields_autoplaced)
-    (property "Reference" "U1" (id 0) (at 53.6575 156.845 0))
-    (property "Value" "XC9572XL-10VQG44C" (id 1) (at 53.6575 159.385 0))
-    (property "Footprint" "Imported:TO_11B1-RK-TP_3MM" (id 2) (at 79.375 173.355 0)
-      (effects (font (size 1.27 1.27)) hide)
-    )
-    (property "Datasheet" "" (id 3) (at 79.375 173.355 0)
-      (effects (font (size 1.27 1.27)) hide)
-    )
-    (property "Reference_1" "IC" (id 4) (at 53.6575 161.925 0))
-    (property "Value_1" "XC9572XL-10VQG44C" (id 5) (at 53.6575 164.465 0))
-    (property "Footprint_1" "QFP80P1200X1200X120-44N" (id 6) (at 74.93 264.465 0)
-      (effects (font (size 1.27 1.27)) (justify left top) hide)
-    )
-    (property "Datasheet_1" "https://componentsearchengine.com/Datasheets/2/XC9572XL-10VQG44C.pdf" (id 7) (at 74.93 364.465 0)
-      (effects (font (size 1.27 1.27)) (justify left top) hide)
-    )
-    (property "Height" "1.2" (id 8) (at 74.93 564.465 0)
-      (effects (font (size 1.27 1.27)) (justify left top) hide)
-    )
-    (property "heisener Part Number" "" (id 9) (at 74.93 664.465 0)
-      (effects (font (size 1.27 1.27)) (justify left top) hide)
-    )
-    (property "heisener Price/Stock" "" (id 10) (at 74.93 764.465 0)
-      (effects (font (size 1.27 1.27)) (justify left top) hide)
-    )
-    (property "Manufacturer_Name" "XILINX" (id 11) (at 74.93 864.465 0)
-      (effects (font (size 1.27 1.27)) (justify left top) hide)
-    )
-    (property "Manufacturer_Part_Number" "XC9572XL-10VQG44C" (id 12) (at 74.93 964.465 0)
-      (effects (font (size 1.27 1.27)) (justify left top) hide)
-    )
-    (pin "1")
-    (pin "10")
-    (pin "11")
-    (pin "12")
-    (pin "13")
-    (pin "14")
-    (pin "15")
-    (pin "16")
-    (pin "17")
-    (pin "18")
-    (pin "19")
-    (pin "2")
-    (pin "20")
-    (pin "21")
-    (pin "22")
-    (pin "23")
-    (pin "24")
-    (pin "25")
-    (pin "26")
-    (pin "27")
-    (pin "28")
-    (pin "29")
-    (pin "3")
-    (pin "30")
-    (pin "31")
-    (pin "32")
-    (pin "33")
-    (pin "34")
-    (pin "35")
-    (pin "36")
-    (pin "37")
-    (pin "38")
-    (pin "39")
-    (pin "4")
-    (pin "40")
-    (pin "41")
-    (pin "42")
-    (pin "43")
-    (pin "44")
-    (pin "5")
-    (pin "6")
-    (pin "7")
-    (pin "8")
-    (pin "9")
-  )
   (symbol (lib_id "Device:R") (at 287.02 172.085 0) (unit 1)
     (in_bom yes) (on_board yes)
@@
     (pin "2")
   )
+  (symbol (lib_id "Imported:XC9572XL-PC44") (at 33.02 164.465 0) (unit 1)
+    (in_bom yes) (on_board yes) (fields_autoplaced)
+    (property "Reference" "U?" (id 0) (at 53.6575 162.56 0))
+    (property "Value" "XC9572XL-PC44" (id 1) (at 53.6575 165.1 0))
+    (property "Footprint" "" (id 2) (at 33.02 164.465 0)
+      (effects (font (size 1.27 1.27)) hide)
+    )
+    (property "Datasheet" "" (id 3) (at 33.02 164.465 0)
+      (effects (font (size 1.27 1.27)) hide)
+    )
+    (pin "1")
+    (pin "10")
+    (pin "11")
+    (pin "12")
+    (pin "13")
+    (pin "14")
+    (pin "15")
+    (pin "16")
+    (pin "17")
+    (pin "18")
+    (pin "19")
+    (pin "2")
+    (pin "20")
+    (pin "21")
+    (pin "22")
+    (pin "23")
+    (pin "24")
+    (pin "25")
+    (pin "26")
+    (pin "27")
+    (pin "28")
+    (pin "29")
+    (pin "3")
+    (pin "30")
+    (pin "31")
+    (pin "32")
+    (pin "33")
+    (pin "34")
+    (pin "35")
+    (pin "36")
+    (pin "37")
+    (pin "38")
+    (pin "39")
+    (pin "4")
+    (pin "40")
+    (pin "41")
+    (pin "42")
+    (pin "43")
+    (pin "44")
+    (pin "5")
+    (pin "6")
+    (pin "7")
+    (pin "8")
+    (pin "9")
+  )
   (symbol (lib_id "power:GND") (at 287.655 95.25 0) (unit 1)
     (in_bom yes) (on_board yes)
@@
     (property "Reference" "U8" (id 0) (at 351.79 27.94 0))
     (property "Value" "MAX6816EUS_T" (id 1) (at 351.79 30.48 0))
-    (property "Footprint" "Package_TO_SOT_SMD:SOT-143_Handsoldering" (id 2) (at 344.805 36.83 0)
+    (property "Footprint" "Package_TO_SOT_SMD:SOT-143R_Reverse_Handsoldering" (id 2) (at 344.805 36.83 0)
       (effects (font (size 1.27 1.27)) (justify bottom) hide)
     )
@@
       (reference "SW1") (unit 1) (value "SW_Push") (footprint "Button_Switch_THT:SW_PUSH_6mm")
     )
-    (path "/223f5043-af9e-431e-83a4-450f66793791"
-      (reference "U1") (unit 1) (value "XC9572XL-10VQG44C") (footprint "Imported:TO_11B1-RK-TP_3MM")
-    )
     (path "/0c317ef6-621d-47c2-9505-4fe082bcdd33"
       (reference "U2") (unit 1) (value "AS6C1008-55PCN") (footprint "Imported:PDIP32_PH_SST_MCH")
@@
     )
     (path "/c87c9639-3b8c-4ff6-a227-4d285f2e5a48"
-      (reference "U8") (unit 1) (value "MAX6816EUS_T") (footprint "Package_TO_SOT_SMD:SOT-143_Handsoldering")
+      (reference "U8") (unit 1) (value "MAX6816EUS_T") (footprint "Package_TO_SOT_SMD:SOT-143R_Reverse_Handsoldering")
     )
     (path "/ab31a195-6c25-48bb-b30b-aa18daeac60d"
@@
       (reference "U10") (unit 1) (value "STM1001LWX6F") (footprint "Imported:SOT-23_STM-L")
     )
+    (path "/498c61a7-be36-43cd-90df-6e60f0c85fa5"
+      (reference "U?") (unit 1) (value "XC9572XL-PC44") (footprint "")
+    )
     (path "/510a45b1-c968-4cb6-8afd-df79c3d13ebe"

Commit message: finished pcb, not checked yet but drc is good
Parts:
- U1: renamed from U?; footprint (none) -> Imported:TO_11B1-RK-TP_3MM
Connections:
- net A19: now also U1.43 (I/O_27); no longer U1.13 (I/O_9)
- net A20: now also U1.40 (I/O/GTS2); no longer U1.14 (I/O_10)
- net A21: now also U1.1 (I/O_1); no longer U1.18 (I/O_11)
- net A22: now also U1.42 (I/O/GTS1); no longer U1.19 (I/O_12)
- net A23: now also U1.33 (I/O_21); no longer U1.20 (I/O_13)
- net AS: now also U1.34 (I/O_22); no longer U1.22 (I/O_14)
- net BRESET: now also U1.19 (I/O_12); no longer U1.2 (I/O_2)
- net CLK: now also U1.6 (I/O/GCK2); no longer U1.7 (I/O/GCK3)
- net DUARTCS: now also U1.3 (I/O_3); no longer U1.42 (I/O/GTS1)
- net DUART_DTACK: now also U1.44 (I/O_28); no longer U1.3 (I/O_3)
- net LDS: now also U1.36 (I/O_24); no longer U1.25 (I/O_16)
- net LED0: now also U1.2 (I/O_2); no longer U1.4 (I/O_4)
- net LED1: now also U1.4 (I/O_4); no longer U1.5 (I/O/GCK1)
- net LED2: now also U1.5 (I/O/GCK1); no longer U1.6 (I/O/GCK2)
- net LED4: now also U1.7 (I/O/GCK3); no longer U1.9 (I/O_6)
- net LED5: now also U1.9 (I/O_6); no longer U1.11 (I/O_7)
- net RAMHCE: now also U1.13 (I/O_9); no longer U1.43 (I/O_27)
- net RAMHCE2: now also U1.11 (I/O_7); no longer U1.44 (I/O_28)
- net RAMHOE: now also U1.14 (I/O_10); no longer U1.40 (I/O/GTS2)
- net RAMLCE2: now also U1.25 (I/O_16); no longer U1.36 (I/O_24)
- net RAMLOE: now also U1.24 (I/O_15); no longer U1.38 (I/O_26)
- net ROMHCE: now also U1.22 (I/O_14); no longer U1.34 (I/O_22)
- net ROMHOE: now also U1.20 (I/O_13); no longer U1.33 (I/O_21)
- net SRESET: now also U1.18 (I/O_11); no longer U1.1 (I/O_1)
- net UDS: now also U1.38 (I/O_26); no longer U1.24 (I/O_15)
Changed lines of the file:
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@@
   (symbol (lib_id "Imported:XC9572XL-PC44") (at 33.02 164.465 0) (unit 1)
     (in_bom yes) (on_board yes) (fields_autoplaced)
-    (property "Reference" "U?" (id 0) (at 53.6575 162.56 0))
+    (property "Reference" "U1" (id 0) (at 53.6575 162.56 0))
     (property "Value" "XC9572XL-PC44" (id 1) (at 53.6575 165.1 0))
-    (property "Footprint" "" (id 2) (at 33.02 164.465 0)
+    (property "Footprint" "Imported:TO_11B1-RK-TP_3MM" (id 2) (at 33.02 164.465 0)
       (effects (font (size 1.27 1.27)) hide)
     )
@@
       (reference "SW1") (unit 1) (value "SW_Push") (footprint "Button_Switch_THT:SW_PUSH_6mm")
     )
+    (path "/498c61a7-be36-43cd-90df-6e60f0c85fa5"
+      (reference "U1") (unit 1) (value "XC9572XL-PC44") (footprint "Imported:TO_11B1-RK-TP_3MM")
+    )
     (path "/0c317ef6-621d-47c2-9505-4fe082bcdd33"
       (reference "U2") (unit 1) (value "AS6C1008-55PCN") (footprint "Imported:PDIP32_PH_SST_MCH")
@@
       (reference "U10") (unit 1) (value "STM1001LWX6F") (footprint "Imported:SOT-23_STM-L")
     )
-    (path "/498c61a7-be36-43cd-90df-6e60f0c85fa5"
-      (reference "U?") (unit 1) (value "XC9572XL-PC44") (footprint "")
-    )
     (path "/510a45b1-c968-4cb6-8afd-df79c3d13ebe"

Commit message: now converts to hex to bin and bin to hex
Parts:
- U8: footprint Package_TO_SOT_SMD:SOT-143R_Reverse_Handsoldering -> Package_TO_SOT_SMD:SOT-143_Handsoldering
Connections:
- net A19: now also U1.35 (I/O_23); no longer U1.43 (I/O_27)
- net A20: now also U1.36 (I/O_24); no longer U1.40 (I/O/GTS2)
- net A21: now also U1.33 (I/O_21); no longer U1.1 (I/O_1)
- net A22: now also U1.34 (I/O_22); no longer U1.42 (I/O/GTS1)
- net A23: now also U1.29 (I/O_20); no longer U1.33 (I/O_21)
- net AS: now also U1.1 (I/O_1); no longer U1.34 (I/O_22)
- net BERR: now also U1.38 (I/O_26); no longer U1.27 (I/O_18)
- net CPLD_DTACK: now also U1.40 (I/O/GTS2); no longer U1.39 (I/O/GSR)
- net HALT: now also U1.39 (I/O/GSR); no longer U1.26 (I/O_17)
- net LDS: now also U1.43 (I/O_27); no longer U1.36 (I/O_24)
- net RAMLCE: now also U1.27 (I/O_18); no longer U1.35 (I/O_23)
- net ROMLCE: now also U1.28 (I/O_19); no longer U1.29 (I/O_20)
- net ROMLOE: now also U1.26 (I/O_17); no longer U1.28 (I/O_19)
- net UDS: now also U1.42 (I/O/GTS1); no longer U1.38 (I/O_26)
Changed lines of the file:
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@@
     (property "Reference" "U8" (id 0) (at 351.79 27.94 0))
     (property "Value" "MAX6816EUS_T" (id 1) (at 351.79 30.48 0))
-    (property "Footprint" "Package_TO_SOT_SMD:SOT-143R_Reverse_Handsoldering" (id 2) (at 344.805 36.83 0)
+    (property "Footprint" "Package_TO_SOT_SMD:SOT-143_Handsoldering" (id 2) (at 344.805 36.83 0)
       (effects (font (size 1.27 1.27)) (justify bottom) hide)
     )
@@
     )
     (path "/c87c9639-3b8c-4ff6-a227-4d285f2e5a48"
-      (reference "U8") (unit 1) (value "MAX6816EUS_T") (footprint "Package_TO_SOT_SMD:SOT-143R_Reverse_Handsoldering")
+      (reference "U8") (unit 1) (value "MAX6816EUS_T") (footprint "Package_TO_SOT_SMD:SOT-143_Handsoldering")
     )
     (path "/ab31a195-6c25-48bb-b30b-aa18daeac60d"
