File: Rev1/KiCAD/MCD/MCD.kicad_pcb (KiCad board)
At the start: 2 copper layers, 196.3 x 114.9 mm, 76 parts, among them J1 DBUS_LOW, J2 DBUS_HIGH, J3 ABUS, J4 POWER, J5 JTAG, J6 Conn_01x02_Male, J7 DUART A, J8 DUART B, SW1 SW_Push, U1 XC9572XL-PC44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

Commit message: added morg files
Routing:
- net A1: track 512.7 -> 509.1 mm
- net A2: track 485.8 -> 482.3 mm
- net A3: track 471.1 -> 468.0 mm
- net A4: track 442.4 -> 439.4 mm
